File: Temporizador Insoladora/Controlador-temporizador/$Controlador-Temporizador Insoladora.sch (KiCad schematic (older format))
At the start: 75 parts, among them P1 ICSP, P2 VAC12V, P3 CARGA, P4 TRANSF, P5 VAC, P6 OPTO, P7 CONN_02X08, P8 OPTO, Q1 BC548, Q2 BC548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

Commit message: Sigo ruteando, falta poco
Connections:
- net VCC: no longer P8.1 (P1), U3.1
- new net: P8.1 (P1), U3.1
Changed lines of the file:
@@
 Wire Wire Line
 	10250 2900 10250 3150
-$Comp
-L VCC #PWR021
-U 1 1 552AC1EA
-P 10250 2750
-F 0 "#PWR021" H 10250 2600 50  0001 C CNN
-F 1 "VCC" H 10250 2900 50  0000 C CNN
-F 2 "" H 10250 2750 60  0000 C CNN
-F 3 "" H 10250 2750 60  0000 C CNN
-	1    10250 2750
-	1    0    0    -1
-$EndComp
 Wire Wire Line
 	10250 2750 10250 2800
@@
 Connection ~ 12250 3400
 $Comp
-L VCC #PWR022
+L VCC #PWR021
 U 1 1 552AD000
 P 2150 3650
-F 0 "#PWR022" H 2150 3500 50  0001 C CNN
+F 0 "#PWR021" H 2150 3500 50  0001 C CNN
 F 1 "VCC" H 2150 3800 50  0000 C CNN
 F 2 "" H 2150 3650 60  0000 C CNN
@@
 $EndComp
 $Comp
-L GND #PWR023
+L GND #PWR022
 U 1 1 552AD006
 P 2150 4150
-F 0 "#PWR023" H 2150 3900 50  0001 C CNN
+F 0 "#PWR022" H 2150 3900 50  0001 C CNN
 F 1 "GND" H 2150 4000 50  0000 C CNN
 F 2 "" H 2150 4150 60  0000 C CNN
@@
 	2150 3650 2150 3750
 $Comp
-L VCC #PWR024
+L VCC #PWR023
 U 1 1 552AD090
 P 1100 4600
-F 0 "#PWR024" H 1100 4450 50  0001 C CNN
+F 0 "#PWR023" H 1100 4450 50  0001 C CNN
 F 1 "VCC" H 1100 4750 50  0000 C CNN
 F 2 "" H 1100 4600 60  0000 C CNN
@@
 $EndComp
 $Comp
-L GND #PWR025
+L GND #PWR024
 U 1 1 552AD096
 P 1100 5100
-F 0 "#PWR025" H 1100 4850 50  0001 C CNN
+F 0 "#PWR024" H 1100 4850 50  0001 C CNN
 F 1 "GND" H 1100 4950 50  0000 C CNN
 F 2 "" H 1100 5100 60  0000 C CNN
@@
 	14050 2950 14200 2950
 $Comp
-L Earth #PWR026
+L Earth #PWR025
 U 1 1 552AE860
 P 14050 3100
-F 0 "#PWR026" H 14050 2850 50  0001 C CNN
+F 0 "#PWR025" H 14050 2850 50  0001 C CNN
 F 1 "Earth" H 14050 2950 50  0001 C CNN
 F 2 "" H 14050 3100 60  0000 C CNN
@@
 $EndComp
 $Comp
-L GND #PWR027
+L GND #PWR026
 U 1 1 552B01E5
 P 7900 6750
-F 0 "#PWR027" H 7900 6500 50  0001 C CNN
+F 0 "#PWR026" H 7900 6500 50  0001 C CNN
 F 1 "GND" H 7900 6600 50  0000 C CNN
 F 2 "" H 7900 6750 60  0000 C CNN
@@
 $EndComp
 $Comp
-L VCC #PWR028
+L VCC #PWR027
 U 1 1 552B0938
 P 7900 5150
-F 0 "#PWR028" H 7900 5000 50  0001 C CNN
+F 0 "#PWR027" H 7900 5000 50  0001 C CNN
 F 1 "VCC" H 7900 5300 50  0000 C CNN
 F 2 "" H 7900 5150 60  0000 C CNN
@@
 	2900 2950 2900 2750
 $Comp
-L GND #PWR029
+L GND #PWR028
 U 1 1 552B5011
 P 3150 2500
-F 0 "#PWR029" H 3150 2250 50  0001 C CNN
+F 0 "#PWR028" H 3150 2250 50  0001 C CNN
 F 1 "GND" H 3150 2350 50  0000 C CNN
 F 2 "" H 3150 2500 60  0000 C CNN
@@
 $EndComp
 $Comp
-L GND #PWR030
+L GND #PWR029
 U 1 1 552AC31E
 P 4000 10450
-F 0 "#PWR030" H 4000 10200 50  0001 C CNN
+F 0 "#PWR029" H 4000 10200 50  0001 C CNN
 F 1 "GND" H 4000 10300 50  0000 C CNN
 F 2 "" H 4000 10450 60  0000 C CNN
@@
 	2000 6000 2000 5750
 $Comp
-L PWR_FLAG #FLG031
+L PWR_FLAG #FLG030
 U 1 1 552BA99D
 P 10050 4700
-F 0 "#FLG031" H 10050 4795 50  0001 C CNN
+F 0 "#FLG030" H 10050 4795 50  0001 C CNN
 F 1 "PWR_FLAG" H 10050 4880 50  0000 C CNN
 F 2 "" H 10050 4700 60  0000 C CNN
@@
 $EndComp
 $Comp
-L GND #PWR032
+L GND #PWR031
 U 1 1 552BAA37
 P 10050 4700
-F 0 "#PWR032" H 10050 4450 50  0001 C CNN
+F 0 "#PWR031" H 10050 4450 50  0001 C CNN
 F 1 "GND" H 10050 4550 50  0000 C CNN
 F 2 "" H 10050 4700 60  0000 C CNN
@@
 $EndComp
 $Comp
-L GND #PWR033
+L GND #PWR032
 U 1 1 552BD498
 P 6450 10450
-F 0 "#PWR033" H 6450 10200 50  0001 C CNN
+F 0 "#PWR032" H 6450 10200 50  0001 C CNN
 F 1 "GND" H 6450 10300 50  0000 C CNN
 F 2 "" H 6450 10450 60  0000 C CNN
@@
 $EndComp
 $Comp
-L GND #PWR034
+L GND #PWR033
 U 1 1 552BDAE3
 P 8900 10450
-F 0 "#PWR034" H 8900 10200 50  0001 C CNN
+F 0 "#PWR033" H 8900 10200 50  0001 C CNN
 F 1 "GND" H 8900 10300 50  0000 C CNN
 F 2 "" H 8900 10450 60  0000 C CNN
@@
 NoConn ~ 5650 2650
 $Comp
-L PWR_FLAG #FLG035
+L PWR_FLAG #FLG034
 U 1 1 552B274E
 P 10500 4700
-F 0 "#FLG035" H 10500 4795 50  0001 C CNN
+F 0 "#FLG034" H 10500 4795 50  0001 C CNN
 F 1 "PWR_FLAG" H 10500 4880 50  0000 C CNN
 F 2 "" H 10500 4700 60  0000 C CNN
@@
 $EndComp
 $Comp
-L Earth #PWR036
+L Earth #PWR035
 U 1 1 552B349E
 P 10500 4700
-F 0 "#PWR036" H 10500 4450 50  0001 C CNN
+F 0 "#PWR035" H 10500 4450 50  0001 C CNN
 F 1 "Earth" H 10500 4550 50  0001 C CNN
 F 2 "" H 10500 4700 60  0000 C CNN
@@
 $EndComp
 $Comp
-L GND #PWR037
+L GND #PWR036
 U 1 1 552BDC57
 P 10550 10450
-F 0 "#PWR037" H 10550 10200 50  0001 C CNN
+F 0 "#PWR036" H 10550 10200 50  0001 C CNN
 F 1 "GND" H 10550 10300 50  0000 C CNN
 F 2 "" H 10550 10450 60  0000 C CNN
@@
 Connection ~ 10250 3000
 $Comp
-L VCC #PWR038
+L VCC #PWR037
 U 1 1 554272CB
 P 8050 3400
-F 0 "#PWR038" H 8050 3250 50  0001 C CNN
+F 0 "#PWR037" H 8050 3250 50  0001 C CNN
 F 1 "VCC" H 8050 3550 50  0000 C CNN
 F 2 "" H 8050 3400 60  0000 C CNN
