File: Temporizador Insoladora/Controlador-temporizador/Controlador-Temporizador Insoladora.kicad_pcb (KiCad board)
At the start: 2 copper layers, 113 x 66 mm, 77 parts, among them P1 ICSP, P2 VAC12V, P3 CARGA, P4 TRANSF, P5 VAC, P6 OPTO, P7 CONN_02X08, P8 OPTO, P9 OPTO, Q1 BC548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

Commit message: Reacomodando controlador
Parts:
- moved C8 11.9 mm to (80.0, 74.9)
Routing:
- net Net-(D2-Pad1): track 18.8 -> 22.6 mm
Other:
- board size 113 x 66 mm -> 99.1 x 66 mm
- net class Pista1.5mm added: clearance 0.8, trace_width 1.5, via_dia 2.5, via_drill 0.7
Changed lines of the file:
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@@
     (links 148)
     (no_connects 0)
-    (area 52.019999 63.449999 165.150001 129.590001)
+    (area 39.56143 58.11 212.89 137.320001)
     (thickness 1.6)
-    (drawings 7)
+    (drawings 6)
     (tracks 345)
     (zones 0)
@@
     (add_net "Net-(C13-Pad2)")
     (add_net "Net-(C4-Pad1)")
-    (add_net "Net-(C8-Pad1)")
     (add_net "Net-(D5-Pad2)")
     (add_net "Net-(D6-Pad1)")
@@
     (add_net VCC)
     (add_net ~MCLR~/VPP)
+  )
+  (net_class Pista1.5mm ""
+    (clearance 0.8)
+    (trace_width 1.5)
+    (via_dia 2.5)
+    (via_drill 0.7)
+    (uvia_dia 0.3)
+    (uvia_drill 0.1)
+    (add_net "Net-(C8-Pad1)")
   )
   (net_class Pista2mm ""
@@
   )
   (module Capacitors_ThroughHole:C_Radial_D10_L16_P5 (layer F.Cu)
-    (at 69.85 81.2 90)
+    (at 80.01 74.93 90)
     (descr "Radial Electrolytic Capacitor 10mm x Length 16mm, Pitch 5mm")
     (tags "Electrolytic Capacitor")
@@
       (net 1 VCC))
   )
-  (dimension 100.33 (width 0.3) (layer Dwgs.User)
-    (gr_text 100,330mm (at 114.935 59.61) (layer Dwgs.User)
+  (dimension 66.04 (width 0.3) (layer Dwgs.User)
+    (gr_text 66,040mm (at 60.88 96.52 90) (layer Dwgs.User)
       (effects (font (size 1.5 1.5) (thickness 0.3)))
     )
-    (feature1 (pts (xy 64.77 63.5) (xy 64.77 58.26)))
-    (feature2 (pts (xy 165.1 63.5) (xy 165.1 58.26)))
-    (crossbar (pts (xy 165.1 60.96) (xy 64.77 60.96)))
-    (arrow1a (pts (xy 64.77 60.96) (xy 65.896504 60.373579)))
-    (arrow1b (pts (xy 64.77 60.96) (xy 65.896504 61.546421)))
-    (arrow2a (pts (xy 165.1 60.96) (xy 163.973496 60.373579)))
-    (arrow2b (pts (xy 165.1 60.96) (xy 163.973496 61.546421)))
-  )
-  (dimension 66.04 (width 0.3) (layer Dwgs.User)
-    (gr_text 66,040mm (at 45.64 96.52 90) (layer Dwgs.User)
+    (feature1 (pts (xy 66.04 63.5) (xy 59.53 63.5)))
+    (feature2 (pts (xy 66.04 129.54) (xy 59.53 129.54)))
+    (crossbar (pts (xy 62.23 129.54) (xy 62.23 63.5)))
+    (arrow1a (pts (xy 62.23 63.5) (xy 62.816421 64.626504)))
+    (arrow1b (pts (xy 62.23 63.5) (xy 61.643579 64.626504)))
+    (arrow2a (pts (xy 62.23 129.54) (xy 62.816421 128.413496)))
+    (arrow2b (pts (xy 62.23 129.54) (xy 61.643579 128.413496)))
+  )
+  (dimension 99.06 (width 0.3) (layer Dwgs.User)
+    (gr_text 99,060mm (at 115.57 59.61) (layer Dwgs.User)
       (effects (font (size 1.5 1.5) (thickness 0.3)))
     )
-    (feature1 (pts (xy 52.07 63.5) (xy 44.29 63.5)))
-    (feature2 (pts (xy 52.07 129.54) (xy 44.29 129.54)))
-    (crossbar (pts (xy 46.99 129.54) (xy 46.99 63.5)))
-    (arrow1a (pts (xy 46.99 63.5) (xy 47.576421 64.626504)))
-    (arrow1b (pts (xy 46.99 63.5) (xy 46.403579 64.626504)))
-    (arrow2a (pts (xy 46.99 129.54) (xy 47.576421 128.413496)))
-    (arrow2b (pts (xy 46.99 129.54) (xy 46.403579 128.413496)))
-  )
-  (dimension 113.03 (width 0.3) (layer Dwgs.User)
-    (gr_text 113,030mm (at 108.585 135.97) (layer Dwgs.User)
-      (effects (font (size 1.5 1.5) (thickness 0.3)))
-    )
-    (feature1 (pts (xy 165.1 129.54) (xy 165.1 137.32)))
-    (feature2 (pts (xy 52.07 129.54) (xy 52.07 137.32)))
-    (crossbar (pts (xy 52.07 134.62) (xy 165.1 134.62)))
-    (arrow1a (pts (xy 165.1 134.62) (xy 163.973496 135.206421)))
-    (arrow1b (pts (xy 165.1 134.62) (xy 163.973496 134.033579)))
-    (arrow2a (pts (xy 52.07 134.62) (xy 53.196504 135.206421)))
-    (arrow2b (pts (xy 52.07 134.62) (xy 53.196504 134.033579)))
-  )
-  (gr_line (start 52.07 129.54) (end 52.07 63.5) (angle 90) (layer Edge.Cuts) (width 0.1))
-  (gr_line (start 165.1 129.54) (end 52.07 129.54) (angle 90) (layer Edge.Cuts) (width 0.1))
+    (feature1 (pts (xy 165.1 63.5) (xy 165.1 58.26)))
+    (feature2 (pts (xy 66.04 63.5) (xy 66.04 58.26)))
+    (crossbar (pts (xy 66.04 60.96) (xy 165.1 60.96)))
+    (arrow1a (pts (xy 165.1 60.96) (xy 163.973496 61.546421)))
+    (arrow1b (pts (xy 165.1 60.96) (xy 163.973496 60.373579)))
+    (arrow2a (pts (xy 66.04 60.96) (xy 67.166504 61.546421)))
+    (arrow2b (pts (xy 66.04 60.96) (xy 67.166504 60.373579)))
+  )
+  (gr_line (start 165.1 129.54) (end 66.04 129.54) (angle 90) (layer Edge.Cuts) (width 0.1))
+  (gr_line (start 66.04 63.5) (end 165.1 63.5) (angle 90) (layer Edge.Cuts) (width 0.1))
+  (gr_line (start 66.04 63.5) (end 66.04 129.54) (angle 90) (layer Edge.Cuts) (width 0.1))
   (gr_line (start 165.1 63.5) (end 165.1 129.54) (angle 90) (layer Edge.Cuts) (width 0.1))
-  (gr_line (start 52.07 63.5) (end 165.1 63.5) (angle 90) (layer Edge.Cuts) (width 0.1))
   (segment (start 86.36 86.36) (end 86.36 88.9) (width 1) (layer B.Cu) (net 1))
   (segment (start 86.36 88.9) (end 87.63 88.9) (width 1) (layer B.Cu) (net 1))
@@
   (segment (start 90.17 111.76) (end 91.44 110.49) (width 1) (layer B.Cu) (net 3))
   (segment (start 90.17 113.03) (end 90.17 111.76) (width 1) (layer B.Cu) (net 3))
-  (segment (start 80.01 88.9) (end 80.01 87.63) (width 1) (layer B.Cu) (net 4))
-  (segment (start 80.01 87.63) (end 77.47 85.09) (width 1) (layer B.Cu) (net 4))
-  (segment (start 77.47 85.09) (end 77.47 81.28) (width 1) (layer B.Cu) (net 4))
-  (segment (start 80.01 88.9) (end 80.01 93.98) (width 1) (layer B.Cu) (net 4))
-  (segment (start 77.47 81.28) (end 69.93 81.28) (width 1) (layer B.Cu) (net 4))
-  (segment (start 69.93 81.28) (end 69.85 81.2) (width 1) (layer B.Cu) (net 4))
+  (segment (start 77.47 81.28) (end 77.47 77.47) (width 1.5) (layer B.Cu) (net 4))
+  (segment (start 77.47 77.47) (end 80.01 74.93) (width 1.5) (layer B.Cu) (net 4))
+  (segment (start 80.09 74.93) (end 80.01 74.85) (width 1) (layer B.Cu) (net 4) (status 30))
+  (segment (start 77.47 86.36) (end 77.47 81.28) (width 1.5) (layer B.Cu) (net 4))
+  (segment (start 80.01 88.9) (end 77.47 86.36) (width 1.5) (layer B.Cu) (net 4))
+  (segment (start 80.01 88.9) (end 80.01 93.98) (width 1.5) (layer B.Cu) (net 4))
   (segment (start 106.68 95.25) (end 106.68 92.71) (width 1) (layer B.Cu) (net 5))
   (segment (start 102.87 87.63) (end 102.87 86.36) (width 1) (layer B.Cu) (net 5))
@@
   (segment (start 113.03 86.36) (end 111.76 86.36) (width 1) (layer B.Cu) (net 10))
   (segment (start 72.39 104.14) (end 80.01 104.14) (width 2) (layer B.Cu) (net 11))
+  (segment (start 80.01 107.95) (end 80.01 104.14) (width 2) (layer B.Cu) (net 11))
+  (segment (start 82.55 110.49) (end 80.01 107.95) (width 2) (layer B.Cu) (net 11))
   (segment (start 86.36 110.49) (end 82.55 110.49) (width 2) (layer B.Cu) (net 11))
-  (segment (start 80.01 107.95) (end 80.01 106.68) (width 2) (layer B.Cu) (net 11))
-  (segment (start 80.01 106.68) (end 80.01 104.14) (width 2) (layer B.Cu) (net 11))
-  (segment (start 82.55 110.49) (end 80.01 107.95) (width 2) (layer B.Cu) (net 11))
+  (segment (start 80.01 107.95) (end 80.01 104.14) (width 2) (layer B.Cu) (net 11))
   (segment (start 72.39 91.44) (end 72.39 93.98) (width 2) (layer B.Cu) (net 12))
   (segment (start 69.85 88.9) (end 72.39 91.44) (width 2) (layer B.Cu) (net 12))
@@
     (polygon
       (pts
-        (xy 165.1 63.5) (xy 52.07 63.5) (xy 52.07 129.54) (xy 165.1 129.54)
+        (xy 165.1 63.5) (xy 66.04 63.5) (xy 66.04 129.54) (xy 165.1 129.54)
       )
     )
