File: Fuente TL2575/Fuente dcdc TL2575.sch (KiCad schematic (older format))
At the start: 12 parts, among them U1 TL2575

Commit message: Terminada Fuente TL2575, y controlador
Parts:
- removed Vin1: CONN_01X02, Sockets_WAGO734:WAGO_734_2pin_Straight_RuggedPads, symbol CONN_01X02
- added C5: 100uF, Capacitors_ThroughHole:C_Radial_D6.3_L11.2_P2.5, symbol CP
- added D2, D3: D, Diodes_ThroughHole:Diode_DO-41_SOD81_Horizontal_RM10, symbol D
- added Vin1: CONN_01X03, Connect:bornier3, symbol CONN_01X03
- Vout1: footprint Sockets_WAGO734:WAGO_734_2pin_Straight_RuggedPads -> Connect:bornier2
Connections:
- net GND: now also C5.2, Vin1.2 (P2)
- net at C1.1, C2.1, U1.16 (VIN): now also D2.2 (K), D3.2 (K)
- net at C3.1, C4.1, L1.2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: now also C5.1
- new net: D2.1 (A), Vin1.1 (P1)
- new net: D3.1 (A), Vin1.3 (P3)
Changed lines of the file:
@@
 LIBS:valves
 LIBS:Kicad-Libreria-Fernando
+LIBS:Fuente dcdc TL2575-cache
 EELAYER 25 0
 EELAYER END
@@
 F 0 "Vout1" H 9000 3600 50  0000 C CNN
 F 1 "CONN_01X02" V 9100 3450 50  0000 C CNN
-F 2 "Sockets_WAGO734:WAGO_734_2pin_Straight_RuggedPads" H 9000 3450 60  0001 C CNN
+F 2 "Connect:bornier2" H 9000 3450 60  0001 C CNN
 F 3 "" H 9000 3450 60  0000 C CNN
 	1    9000 3450
 	1    0    0    -1
-$EndComp
-$Comp
-L CONN_01X02 Vin1
-U 1 1 551AF1FF
-P 1850 3400
-F 0 "Vin1" H 1800 3600 50  0000 C CNN
-F 1 "CONN_01X02" V 1950 3400 50  0000 C CNN
-F 2 "Sockets_WAGO734:WAGO_734_2pin_Straight_RuggedPads" H 1850 3400 60  0001 C CNN
-F 3 "" H 1850 3400 60  0000 C CNN
-	1    1850 3400
-	-1   0    0    -1
 $EndComp
 Wire Wire Line
@@
 	9650 4700 9650 4600
 Wire Wire Line
-	2250 3700 3600 3700
+	1500 3700 3600 3700
 Wire Wire Line
 	2250 3100 3600 3100
 Wire Wire Line
-	2250 3100 2250 3350
-Wire Wire Line
-	2250 3450 2250 3700
-Wire Wire Line
-	2250 3350 2050 3350
-Wire Wire Line
-	2050 3450 2250 3450
+	2250 3100 2250 3550
+Wire Wire Line
+	1950 3350 2250 3350
+$Comp
+L CONN_01X03 Vin1
+U 1 1 5564AF0F
+P 1050 3450
+F 0 "Vin1" H 1050 3650 50  0000 C CNN
+F 1 "CONN_01X03" V 1150 3450 50  0000 C CNN
+F 2 "Connect:bornier3" H 1050 3450 60  0001 C CNN
+F 3 "" H 1050 3450 60  0000 C CNN
+	1    1050 3450
+	-1   0    0    -1
+$EndComp
+$Comp
+L D D2
+U 1 1 5564B16C
+P 1800 3350
+F 0 "D2" H 1800 3450 50  0000 C CNN
+F 1 "D" H 1800 3250 50  0000 C CNN
+F 2 "Diodes_ThroughHole:Diode_DO-41_SOD81_Horizontal_RM10" H 1800 3350 60  0001 C CNN
+F 3 "" H 1800 3350 60  0000 C CNN
+	1    1800 3350
+	1    0    0    -1
+$EndComp
+$Comp
+L D D3
+U 1 1 5564B2C0
+P 1800 3550
+F 0 "D3" H 1800 3650 50  0000 C CNN
+F 1 "D" H 1800 3450 50  0000 C CNN
+F 2 "Diodes_ThroughHole:Diode_DO-41_SOD81_Horizontal_RM10" H 1800 3550 60  0001 C CNN
+F 3 "" H 1800 3550 60  0000 C CNN
+	1    1800 3550
+	1    0    0    -1
+$EndComp
+Wire Wire Line
+	1250 3550 1650 3550
+Wire Wire Line
+	1250 3350 1650 3350
+Wire Wire Line
+	2250 3550 1950 3550
+Connection ~ 2250 3350
+Wire Wire Line
+	1250 3450 1500 3450
+Wire Wire Line
+	1500 3450 1500 3700
+$Comp
+L CP C5
+U 1 1 5565CBDE
+P 6700 3900
+F 0 "C5" H 6725 4000 50  0000 L CNN
+F 1 "100uF" H 6725 3800 50  0000 L CNN
+F 2 "Capacitors_ThroughHole:C_Radial_D6.3_L11.2_P2.5" H 6738 3750 30  0001 C CNN
+F 3 "" H 6700 3900 60  0000 C CNN
+	1    6700 3900
+	1    0    0    -1
+$EndComp
+Wire Wire Line
+	6700 3750 6700 3400
+Connection ~ 6700 3400
+Wire Wire Line
+	6700 4050 6700 4500
+Connection ~ 6700 4500
 $EndSCHEMATC
