File: Fuente TL2575-V2/Fuente dcdc TL2575-V2.sch (KiCad schematic (older format))
At the start: 14 parts, among them U1 TL2575

Commit message: Modificando la version 2 de la fuente TL2575
Parts:
- Vin1: value CONN_01X03 -> VIN
- Vout1: value CONN_01X02 -> VOUT
Changed lines of the file:
@@
 P 9000 3450
 F 0 "Vout1" H 9000 3600 50  0000 C CNN
-F 1 "CONN_01X02" V 9100 3450 50  0000 C CNN
+F 1 "VOUT" V 9100 3450 50  0000 C CNN
 F 2 "Connect:bornier2" H 9000 3450 60  0001 C CNN
 F 3 "" H 9000 3450 60  0000 C CNN
@@
 P 1050 3450
 F 0 "Vin1" H 1050 3650 50  0000 C CNN
-F 1 "CONN_01X03" V 1150 3450 50  0000 C CNN
+F 1 "VIN" V 1150 3450 50  0000 C CNN
 F 2 "Connect:bornier3" H 1050 3450 60  0001 C CNN
 F 3 "" H 1050 3450 60  0000 C CNN

Commit message: Finalizando TL2575-V2
Parts:
- added C6: 100nF, Capacitors_ThroughHole:C_Disc_D3_P2.5, symbol C
Connections:
- net GND: now also C6.2
- net at C3.1, C4.1, C5.1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: now also C6.1
Other:
- moved on the sheet: C5
Changed lines of the file:
@@
 	7400 4500 7400 4000
 Wire Wire Line
-	7000 3700 7000 3400
+	7000 3400 7000 3700
 Wire Wire Line
 	6600 3400 8800 3400
@@
 L CP C5
 U 1 1 5565CBDE
-P 6700 3900
-F 0 "C5" H 6725 4000 50  0000 L CNN
-F 1 "100uF" H 6725 3800 50  0000 L CNN
-F 2 "Capacitors_ThroughHole:C_Radial_D6.3_L11.2_P2.5" H 6738 3750 30  0001 C CNN
-F 3 "" H 6700 3900 60  0000 C CNN
-	1    6700 3900
-	1    0    0    -1
-$EndComp
-Wire Wire Line
-	6700 3750 6700 3400
+P 6700 3850
+F 0 "C5" H 6725 3950 50  0000 L CNN
+F 1 "100uF" H 6725 3750 50  0000 L CNN
+F 2 "Capacitors_ThroughHole:C_Radial_D6.3_L11.2_P2.5" H 6738 3700 30  0001 C CNN
+F 3 "" H 6700 3850 60  0000 C CNN
+	1    6700 3850
+	1    0    0    -1
+$EndComp
+Wire Wire Line
+	6700 3700 6700 3400
 Connection ~ 6700 3400
 Wire Wire Line
-	6700 4050 6700 4500
+	6700 4000 6700 4500
 Connection ~ 6700 4500
 Wire Wire Line
 	8300 3700 8300 3400
+$Comp
+L C C6
+U 1 1 55689F71
+P 8600 3900
+F 0 "C6" H 8625 4000 50  0000 L CNN
+F 1 "100nF" H 8625 3800 50  0000 L CNN
+F 2 "Capacitors_ThroughHole:C_Disc_D3_P2.5" H 8638 3750 30  0001 C CNN
+F 3 "" H 8600 3900 60  0000 C CNN
+	1    8600 3900
+	1    0    0    -1
+$EndComp
+Wire Wire Line
+	8600 3750 8600 3400
+Wire Wire Line
+	8600 3400 8650 3400
+Connection ~ 8650 3400
+Wire Wire Line
+	8600 4050 8600 4500
+Connection ~ 8600 4500
 $EndSCHEMATC
